File: reflower.kicad_sch (KiCad schematic)
At the start: 49 parts, among them J1 Screw_Terminal_01x02, J2 Screw_Terminal_01x02, J3 Barrel_Jack, Q1 IRG4PF50W, U1 MAX31855KASA+T, U2 NCP1117-3.3, U3 STM32L010C6T6, U4 ZXGD3006E6, U5 4N25

Commit message: Revisions
Parts:
- removed C9: 10uF, Capacitor_THT:CP_Radial_D5.0mm_P2.00mm, symbol Device:C_Polarized_Small
- removed D3: 1N4007, Diode_THT:D_DO-41_SOD81_P10.16mm_Horizontal, symbol Diode:1N4007
- removed J3: Barrel_Jack, symbol Connector:Barrel_Jack
- removed R12: 10K, symbol Device:R_Small_US
- added D2: 1N4007, Diode_THT:D_DO-41_SOD81_P10.16mm_Horizontal, symbol Diode:1N4007
- added J4: Screw_Terminal_01x02, symbol Connector:Screw_Terminal_01x02
- added R2: 1K, Resistor_SMD:R_0603_1608Metric, symbol Device:R_Small_US
- C5: renamed from C7; value 10uF -> 1uF
- C6: renamed from C8; value 1uF -> 10uF
- D1: value B380C2300-1500B -> B380C2300
- renumbered C11 to C10, C12 to C11, C13 to C12, C14 to C13, C15 to C14, C5 to C7, C6 to C8, C10 to C9, J2 to J3, R9 to R10, R10 to R11, R11 to R12, R2 to R3, R3 to R4, R4 to R5, R5 to R6, R6 to R7, R7 to R8, R8 to R9
Connections:
- net GND: now also R2.2; no longer D1.1 (-), R1.2
- net GNDPWR: now also D1.1 (-), Q1.3 (E); no longer D1.4, J1.2 (Pin_2)
- net VSS: now also J4.2 (Pin_2)
- net at Q1.1 (G), R12.1: now also D2.2 (A)
- net at Q1.2 (C): now also J4.1 (Pin_1)
- net at R12.2, U4.4 (SINK), U4.6 (SRC): now also D2.1 (K)
- new net: R1.2, R2.1
- new net Earth: D1.4, J1.2 (Pin_2)
Other:
- note added: "Load Power"
- note added: "Logic Power"
- note added: "Oven Load"
- note removed: "External safe DC power source is needed for now, until can use mains for logic supply."
- moved on the sheet: C1, C10, C2, C3, C4, C5, C6, C7, C8, C9, D1, DZ1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
